File: S4A_Board/Arduino_ESP.kicad_pcb (KiCad board)
At the start: 4 copper layers, 68.8 x 53.3 mm, 35 parts, among them IC1 ESP32-WROVER, IC2 PDTC, IC3 PDTC, J1 Digitali1, J2 Digitali2, J3 Analogici, J4 Conn_01x07_Male, J5 Aux, J6 USB_C, SW1 RESET, U1 CH340C, U2 AP3211

Commit message: correzione
Routing:
- net RESET: vias 2 -> 3
Changed lines of the file:
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@@
+	)
+	(segment
+		(start 142.3162 97.0534)
+		(end 142.3162 95.9104)
+		(width 0.4)
+		(layer "F.Cu")
+		(net 9)
 	)
 	(segment
@@
 	)
 	(segment
-		(start 128.2076 65.7744)
-		(end 128.2192 65.786)
+		(start 142.3162 95.9104)
+		(end 142.3162 95.885)
 		(width 0.4)
 		(layer "F.Cu")
@@
 	)
 	(segment
-		(start 142.3162 97.0534)
-		(end 142.3162 95.885)
+		(start 128.2076 65.7744)
+		(end 128.2192 65.786)
 		(width 0.4)
 		(layer "F.Cu")
@@
 		(width 0.4)
 		(layer "F.Cu")
+		(net 9)
+	)
+	(via
+		(at 142.3162 95.9104)
+		(size 0.8)
+		(drill 0.4)
+		(layers "F.Cu" "B.Cu")
 		(net 9)
 	)
@@
 	)
 	(segment
-		(start 142.2908 89.7128)
-		(end 145.8976 86.106)
-		(width 0.4)
-		(layer "In2.Cu")
-		(net 9)
-	)
-	(segment
-		(start 148.16 103.456)
-		(end 142.2908 97.5868)
-		(width 0.4)
-		(layer "In2.Cu")
-		(net 9)
-	)
-	(segment
-		(start 142.2908 97.5868)
-		(end 142.2908 95.8596)
-		(width 0.4)
-		(layer "In2.Cu")
-		(net 9)
-	)
-	(segment
-		(start 142.2908 95.8596)
-		(end 142.2908 89.7128)
+		(start 142.3162 97.6122)
+		(end 142.3162 89.6874)
 		(width 0.4)
 		(layer "In2.Cu")
@@
 		(width 0.4)
 		(layer "In2.Cu")
+		(net 9)
+	)
+	(segment
+		(start 142.3162 89.6874)
+		(end 145.8976 86.106)
+		(width 0.4)
+		(layer "In2.Cu")
+		(net 9)
+	)
+	(segment
+		(start 148.16 103.456)
+		(end 142.3162 97.6122)
+		(width 0.4)
+		(layer "In2.Cu")
